Commit message: Pre-commit

File: moveitpy_simple/moveit_configs_utils/test/robot.urdf.xacro (robot description, xacro)
@@ -1,12 +1,12 @@
-<?xml version="1.0" ?>
+<?xml version="1.0"?>
 <robot xmlns:xacro="http://www.ros.org/wiki/xacro">
   <xacro:macro name="robot" params="test_robot number postfix">
     <robot name="$(arg test_robot)">
-      <link name="base" />
-      <link name="link_${postfix}" />
+      <link name="base"/>
+      <link name="link_${postfix}"/>
       <joint name="base_to_link_${postfix}" type="fixed">
-        <parent link="base" />
-        <child link="link_${postfix}" />
-        <origin xyz="0 ${number} 0" />
+        <parent link="base"/>
+        <child link="link_${postfix}"/>
+        <origin xyz="0 ${number} 0"/>
       </joint>
     </robot>
@@ -15,4 +15,4 @@
   <xacro:arg name="number" default="testing_number"/>
   <xacro:arg name="postfix" default="testing_postfix"/>
-  <xacro:robot test_robot="$(arg test_robot)" number="$(arg number)" postfix="$(arg postfix)" />
+  <xacro:robot test_robot="$(arg test_robot)" number="$(arg number)" postfix="$(arg postfix)"/>
 </robot>
